File: hardware/0.2/macro4.sch (KiCad schematic (older format))
At the start: 29 parts, among them J1 USB_C_Receptacle_USB2.0, Q1 BSS138, SW1 SIDE, SW2 SIDE, SW3 CHERRY_MX, SW5 CHERRY_MX, SW6 CHERRY_MX, SW7 Rotary_Encoder_MX, U1 AP2112K-3.3, U2 STM32F072C8Tx

Commit message: added second encoder, fixed panelisation script
Parts:
- removed SW6: CHERRY_MX, josh-keyboard:MX_KEYSWITCH, symbol Switch:SW_Push
- added SW4: Rotary_Encoder_MX, josh-keyboard:MX_KEYSWITCH_ENCODER, symbol Device:Rotary_Encoder_Switch
- LOGO1: footprint josh-logos:josh-johnson-logo-11x2 -> josh-logos:josh-johnson-logo-17x3
- R1, R2: footprint Resistor_SMD:R_0603_1608Metric_Pad1.05x0.95mm_HandSolder -> Resistor_SMD:R_0603_1608Metric
Connections:
- net +3V3: now also RN1.1; no longer RN1.8
- net GND: now also SW4.C, SW4.S2
- net KEY_1: now also SW7.S1, U2.37 (PA14); no longer U2.30 (PA9)
- net KEY_2: now also U2.29 (PA8), SW4.S1; no longer SW7.S1, U2.37 (PA14)
- net nRST: now also RN1.8; no longer RN1.1
- net ENC_2_A: now reaches U2.19 (PB1)
- net ENC_2_A: now also SW4.A
- net ENC_2_B: now reaches U2.20 (PB2)
- net ENC_2_B: now also SW4.B
- net ENC_A renamed ENC_1_A
- net ENC_B renamed ENC_1_B
- no-connect marks 31 -> 29
Other:
- moved on the sheet: SW7
